File: PCB/Test/Test.kicad_sch (KiCad schematic)
At the start: 16 parts, among them J1 USB-C, J2 USB-C, J3 USB-C, J4 USB-C, J5 USB-C, J6 USB-C, J7 USB-C, J8 USB-C, U1 ESP32-PICO-MINI-02, U2 ESP32-PICO-MINI-02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

Commit message: rotate direction
Parts:
- added J9: Conn_01x04, RevK:JLC-PinHeader_1x04_P2.54mm_Right, symbol Connector_Generic:Conn_01x04
Changed lines of the file:
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@@
     (pin "9")
+  )
+  (symbol (lib_id "Connector_Generic:Conn_01x04") (at 60.96 149.86 0) (unit 1)
+    (in_bom yes) (on_board yes) (fields_autoplaced)
+    (property "Reference" "J9" (id 0) (at 62.992 150.2953 0)
+      (effects (font (size 1.27 1.27)) (justify left))
+    )
+    (property "Value" "Conn_01x04" (id 1) (at 62.992 152.8322 0)
+      (effects (font (size 1.27 1.27)) (justify left))
+    )
+    (property "Footprint" "RevK:JLC-PinHeader_1x04_P2.54mm_Right" (id 2) (at 60.96 149.86 0)
+      (effects (font (size 1.27 1.27)) hide)
+    )
+    (property "Datasheet" "~" (id 3) (at 60.96 149.86 0)
+      (effects (font (size 1.27 1.27)) hide)
+    )
+    (pin "1")
+    (pin "2")
+    (pin "3")
+    (pin "4")
   )
   (symbol (lib_id "RevK:ESP32-PICO-MINI-02") (at 196.85 130.175 0) (unit 1)
@@
       (reference "J8") (unit 1) (value "USB-C") (footprint "RevK:USC16-TR-Round")
     )
+    (path "/2010f84f-8452-46e0-84aa-faa2502312d1"
+      (reference "J9") (unit 1) (value "Conn_01x04") (footprint "RevK:JLC-PinHeader_1x04_P2.54mm_Right")
+    )
     (path "/acef3704-d21e-45df-8313-4c7db53fd2c9"

Commit message: Updated test case
Parts:
- removed J2, J3: USB-C, RevK:USC16-TR-Round, symbol RevK:USB-C
- removed U1, U8: ESP32-PICO-MINI-02, RevK:ESP32-PICO-MINI-02, symbol RevK:ESP32-PICO-MINI-02
- added J10: Conn_01x05, RevK:PTSM-HH-5-RA-P, symbol Connector_Generic:Conn_01x05
- added J11: Conn_01x05, RevK:PTSM-HH-5-RA, symbol Connector_Generic:Conn_01x05
- added J12: Conn_01x05, RevK:PTSM-HH-5-RA-P-SMD, symbol Connector_Generic:Conn_01x05
